File: LineOut.kicad_pcb (KiCad board)
At the start: 2 copper layers, 15.2 x 101.6 mm, 9 parts, among them J1 Left, J2 Right, J3 Line Out

Commit message: Upgraded to KiCad 5.02.
Parts:
- J1: value Left -> AudioJack2_SwitchT
- J2: value Right -> AudioJack3; footprint Local:PJ398SM -> Local:PJ366ST
- J3: value Line Out -> AudioJack2_SwitchT; footprint Local:PJ366ST -> Local:PJ398SM
- R2: value 10k -> 1k
- R3: value 1k -> 10k
- moved J3 61.0 mm to (75.9, 96.5), turned to 0 degrees
- moved J2 61.0 mm to (76.2, 157.5), turned to 180 degrees
Connections:
- J1 pad TN: Net-(J1-PadTN) -> GND
- J2 pad T: Net-(J2-PadT) -> Net-(C1-Pad1)
- J3 pad T: Net-(C1-Pad1) -> Net-(J3-PadT)
- R2 pad 1: Net-(C2-Pad2) -> GND
- R2 pad 2: Net-(J2-PadT) -> Net-(C1-Pad2)
- R3 pad 1: GND -> Net-(C2-Pad2)
- R3 pad 2: Net-(C1-Pad2) -> Net-(J3-PadT)
Routing:
- net Net-(J2-PadT): track 60.8 -> 0.00 mm, vias 4 -> 0
- net Net-(C1-Pad2): track 53.3 -> 114.1 mm, vias 0 -> 4
